Commit message: feat: 统一传感器外参与融合参考点
以 robot_description 和 URDF 集中管理 LiDAR、IMU、GPS 静态外参。

通过 TF 完成 FAST-LIO 与 GPS 杆臂补偿，并同步 GPS 航向观测。

新增统一启动、隔离回放入口以及局部和全局路径输出。

File: config/urdf/robot.urdf (robot description, URDF)
Before this commit: robot robot_gps_localization, 4 links, 3 joints
Links:
- added link livox_imu; visual sphere radius=0.025
Joints:
- removed joint base_link_to_livox_frame
- added joint base_link_to_livox_imu: type fixed, parent base_link, child livox_imu, origin xyz=0 0 0 rpy=0 0 0
- added joint livox_imu_to_livox_frame: type fixed, parent livox_imu, child livox_frame, origin xyz=-0.011000 -0.023290 0.044120 rpy=0 0 0
